Commit message: finish urdf & tasted

File: diff_robot/urdf/chassis.xacro (robot description, xacro)
@@ -4,17 +4,18 @@
     <link name="chassis_link">
         <visual>
-            <origin xyz="0.0 0.0 0.075" rpy="0.0 0.0 0.0"/>
+            <origin xyz="0.0 0.0 0.0" rpy="0.0 0.0 0.0"/>
             <geometry>
-                <cylinder radius="0.15" length="0.15"/>
+                <cylinder radius="0.210" length="0.15"/>
             </geometry>
+            <material name="white"/>
         </visual>
         <collision>
-            <origin xyz="0.0 0.0 0.075" rpy="0.0 0.0 0.0"/>
+            <origin xyz="0.0 0.0 0.0" rpy="0.0 0.0 0.0"/>
             <geometry>
-                <cylinder radius="0.15" length="0.15"/>
+                <cylinder radius="0.210" length="0.15"/>
             </geometry>
         </collision>
-        <xacro:inertial_cylinder mass="4" length="0.15" radius="0.15">
-            <origin xyz="0.0 0.0 0.075" rpy="0.0 0.0 0.0"/>
+        <xacro:inertial_cylinder mass="4" length="0.15" radius="0.210">
+            <origin xyz="0.0 0.0 0.0" rpy="0.0 0.0 0.0"/>
         </xacro:inertial_cylinder>
     </link>
@@ -23,5 +24,8 @@
         <parent link="base_link"/>
         <child link="chassis_link"/>
-        <origin xyz="0.05 0.0 0.0" rpy="0.0 0.0 0.0"/>
+        <origin xyz="0.03 0.0 0.0575" rpy="0.0 0.0 0.0"/>
     </joint>
+    <gazebo reference="chassis_link">
+        <material> Gazebo/White</material>
+    </gazebo>
 </robot>

File: diff_robot/urdf/robot.urdf.xacro (robot description, xacro)
@@ -2,5 +2,11 @@
 <robot xmlns:xacro="https://www.ros.org/wiki/xacro" name="diff_robot">
     <xacro:include filename="inertial_macros.xacro"/>
+    <xacro:include filename="properties.xacro"/>
     <xacro:include filename="chassis.xacro"/>
+    <xacro:include filename="wheels.xacro"/>
+    <xacro:include filename="caster_wheel.xacro"/>
+    <xacro:include filename="lidar.xacro"/>
+    <xacro:include filename="imu.xacro"/>
+    <xacro:include filename="gazebo_control.xacro"/>
     <link name="base_link"/>
 </robot>

Commit message: Mapping_Finish

File: diff_robot/urdf/chassis.xacro (robot description, xacro)
@@ -6,5 +6,5 @@
             <origin xyz="0.0 0.0 0.0" rpy="0.0 0.0 0.0"/>
             <geometry>
-                <cylinder radius="0.210" length="0.15"/>
+                <cylinder radius="${chassis_radius}" length="${chassis_height}"/>
             </geometry>
             <material name="white"/>
@@ -13,8 +13,8 @@
             <origin xyz="0.0 0.0 0.0" rpy="0.0 0.0 0.0"/>
             <geometry>
-                <cylinder radius="0.210" length="0.15"/>
+                <cylinder radius="${chassis_radius}" length="${chassis_height}"/>
             </geometry>
         </collision>
-        <xacro:inertial_cylinder mass="4" length="0.15" radius="0.210">
+        <xacro:inertial_cylinder mass="4" length="${chassis_height}" radius="${chassis_radius}">
             <origin xyz="0.0 0.0 0.0" rpy="0.0 0.0 0.0"/>
         </xacro:inertial_cylinder>
@@ -25,4 +25,6 @@
         <child link="chassis_link"/>
         <origin xyz="0.03 0.0 0.0575" rpy="0.0 0.0 0.0"/>
+    <!--In a URDF joint, the <origin> tag defines the pose of the child link relative to
+    the parent link's coordinate frame. so move from parent to the child-->
     </joint>
     <gazebo reference="chassis_link">

File: diff_robot/urdf/robot.urdf.xacro (robot description, xacro)
@@ -10,3 +10,8 @@
     <xacro:include filename="gazebo_control.xacro"/>
     <link name="base_link"/>
+    <link name="base_footprint"/>
+    <joint name="base_footprint_joint" type="fixed">
+        <parent link="base_link"/>
+        <child link="base_footprint"/>
+    </joint>
 </robot>

Commit message: edits_for_TFtree_refining

File: diff_robot/urdf/chassis.xacro (robot description, xacro)
@@ -8,5 +8,5 @@
                 <cylinder radius="${chassis_radius}" length="${chassis_height}"/>
             </geometry>
-            <material name="white"/>
+            <material name="green"/>
         </visual>
         <collision>
@@ -25,9 +25,9 @@
         <child link="chassis_link"/>
         <origin xyz="0.03 0.0 0.0575" rpy="0.0 0.0 0.0"/>
-    <!--In a URDF joint, the <origin> tag defines the pose of the child link relative to
+        <!--In a URDF joint, the <origin> tag defines the pose of the child link relative to
     the parent link's coordinate frame. so move from parent to the child-->
     </joint>
     <gazebo reference="chassis_link">
-        <material> Gazebo/White</material>
+        <material> Gazebo/Green</material>
     </gazebo>
 </robot>

File: diff_robot/urdf/gazebo_control.xacro (robot description, xacro)
@@ -1,26 +1,33 @@
 <?xml version="1.0"?>
 <robot xmlns:xacro="http://www.ros.org/wiki/xacro" >
-      <gazebo>
-  <plugin name="diff_drive" filename="libgazebo_ros_diff_drive.so">
-    <ros>
-      <remapping>joint_states:=/joint_states</remapping>
-      <remapping>odom:=/odom</remapping>
-    </ros>
-    <update_rate>30</update_rate>
-    <left_joint>left_wheel_joint</left_joint>
-    <right_joint>right_wheel_joint</right_joint>
-    <wheel_separation>0.2983</wheel_separation>
-    <wheel_diameter>0.065</wheel_diameter>
-    <max_wheel_torque>20</max_wheel_torque>
-    <max_wheel_acceleration>1.0</max_wheel_acceleration>
-    <odometry_frame>odom</odometry_frame>
-    <robot_base_frame>base_link</robot_base_frame>
-    <publish_odom>true</publish_odom>
-    <publish_odom_tf>true</publish_odom_tf>
-    <publish_wheel_tf>true</publish_wheel_tf>
-    <publish_wheel_joint_state>true</publish_wheel_joint_state>
-    <odometry_topic>odom</odometry_topic>
-    <command_topic>cmd_vel</command_topic>
-  </plugin>
-</gazebo>
+  <gazebo>
+    <plugin name="diff_drive" filename="libgazebo_ros_diff_drive.so">
+      <ros>
+        <remapping>odom:=/odom</remapping>
+      </ros>
+      <update_rate>30</update_rate>
+      <left_joint>left_wheel_joint</left_joint>
+      <right_joint>right_wheel_joint</right_joint>
+      <wheel_separation>0.2983</wheel_separation>
+      <wheel_diameter>0.065</wheel_diameter>
+      <max_wheel_torque>20</max_wheel_torque>
+      <max_wheel_acceleration>1.0</max_wheel_acceleration>
+      <odometry_frame>odom</odometry_frame>
+      <robot_base_frame>base_footprint</robot_base_frame>
+      <publish_odom>true</publish_odom>
+      <publish_odom_tf>false</publish_odom_tf>
+      <publish_wheel_tf>false</publish_wheel_tf>
+      <publish_wheel_joint_state>true</publish_wheel_joint_state>
+      <odometry_topic>odom</odometry_topic>
+      <command_topic>cmd_vel</command_topic>
+    </plugin>
+    <plugin name="joint_state_publisher" filename="libgazebo_ros_joint_state_publisher.so">
+      <ros>
+        <remapping>~/out:=joint_states</remapping>
+      </ros>
+      <update_rate>30</update_rate>
+      <joint_name>left_wheel_joint</joint_name>
+      <joint_name>right_wheel_joint</joint_name>
+    </plugin>
+  </gazebo>
 </robot>

File: diff_robot/urdf/imu.xacro (robot description, xacro)
@@ -7,5 +7,5 @@
           <box size="0.01556012 0.02026185 0.00254"/>
       </geometry>
-      <material name="Red"/>
+      <material name="red"/>
      </visual>
   </link>
@@ -16,6 +16,6 @@
     <child link="imu_frame"/>
   </joint>
-<!--IMU_Plugin-->
-  <gazebo reference="imu_frame">
+<!-- IMU_Plugin -->
+  <!-- <gazebo reference="imu_frame">
     <gravity>true</gravity>
     <sensor name="imu_sensor" type="imu">
@@ -36,4 +36,18 @@
       <pose>0 0 0 0 0 0</pose>
     </sensor>
+  </gazebo> -->
+  <gazebo reference="imu_frame">
+    <gravity>true</gravity>
+    <sensor name="imu_sensor" type="imu">
+      <always_on>true</always_on>
+      <update_rate>100</update_rate>
+      <visualize>true</visualize>
+      <plugin filename="libgazebo_ros_imu_sensor.so" name="imu_plugin">
+        <ros>
+          <remapping>~/out:=imu</remapping>
+        </ros>
+        <initial_orientation_as_reference>false</initial_orientation_as_reference>
+      </plugin>
+    </sensor>
   </gazebo>
   <gazebo reference="imu_frame">

File: diff_robot/urdf/lidar.xacro (robot description, xacro)
@@ -38,5 +38,6 @@
             <plugin name="laser_controller" filename="libgazebo_ros_ray_sensor.so">
                 <ros>
-                    <argument>~/out:=scan</argument>
+                    <!-- <argument>~/out:=scan</argument> -->
+                     <remapping>~/out:=scan</remapping>
                 </ros>
                 <output_type>sensor_msgs/LaserScan</output_type>

File: diff_robot/urdf/robot.urdf.xacro (robot description, xacro)
@@ -12,6 +12,7 @@
     <link name="base_footprint"/>
     <joint name="base_footprint_joint" type="fixed">
-        <parent link="base_link"/>
-        <child link="base_footprint"/>
+        <parent link="base_footprint"/>
+        <child link="base_link"/>
+        <origin xyz="0 0 0.0325" rpy="0 0 0"/>
     </joint>
 </robot>

Commit message: urdf_dimention_edit

File: diff_robot/urdf/chassis.xacro (robot description, xacro)
@@ -24,5 +24,5 @@
         <parent link="base_link"/>
         <child link="chassis_link"/>
-        <origin xyz="0.03 0.0 0.0575" rpy="0.0 0.0 0.0"/>
+        <origin xyz="0.04124 0.0 0.0525" rpy="0.0 0.0 0.0"/>
         <!--In a URDF joint, the <origin> tag defines the pose of the child link relative to
     the parent link's coordinate frame. so move from parent to the child-->

File: diff_robot/urdf/properties.xacro (robot description, xacro)
@@ -4,10 +4,10 @@
 <!-- Chassis-->
 <xacro:property name="chassis_height" value="0.15"/>
-<xacro:property name="chassis_radius" value="0.210"/>
+<xacro:property name="chassis_radius" value="0.213"/>
 <xacro:property name="chassis_mass" value="4.0"/>
 <!-- Wheels-->
-<xacro:property name="wheel_offset_x" value="-0.03"/>
-<xacro:property name="wheel_offset_y" value="0.14915"/>
-<xacro:property name="wheel_offset_z" value="-0.0575"/>
+<xacro:property name="wheel_offset_x" value="-0.04124"/>
+<xacro:property name="wheel_offset_y" value="0.14955"/>
+<xacro:property name="wheel_offset_z" value="-0.0525"/>
 <xacro:property name="wheel_thickness" value="0.027"/>
 <xacro:property name="wheel_radius" value="0.0325"/>
